File: hardware/pcb-main/pcb.kicad_pcb (KiCad board)
At the start: 2 copper layers, 276.2 x 71.4 mm, 105 parts, among them P1 USB, SW1 SW_PUSH, U00 MX-DI, U01 MX-DI, U010 MX-DI, U011 MX-DI, U012 MX-DI, U02 MX-DI, U03 MX-DI, U04 MX-DI, U05 MX-DI, U06 MX-DI, U07 MX-DI, U08 MX-DI, U09 MX-DI, U1 ATmega32U4, U10 MX-DI, U11 MX-DI, U110 MX-DI, U111 MX-DI, U112 MX-DI, U113 MX-DI, U12 MX-DI, U13 MX-DI, U14 MX-DI, U15 MX-DI, U16 MX-DI, U17 MX-DI, U18 MX-DI, U19 MX-DI, U20 MX-DI, U21 MX-DI, U210 MX-DI, U211 MX-DI, U212 MX-DI, U213 MX-DI, U22 MX-DI, U23 MX-DI, U24 MX-DI, U25 MX-DI, U26 MX-DI, U27 MX-DI, U28 MX-DI, U29 MX-DI, U30 MX-DI, U31 MX-DI, U310 MX-DI, U311 MX-DI, U312 MX-DI, U313 MX-DI, U32 MX-DI, U34 MX-DI, U35 MX-DI, U37 MX-DI, U38 MX-DI, Y1 HC49S

Commit message: Reduce PCB width
Other:
- board size 276.2 x 71.4 mm -> 274.9 x 71.4 mm
Changed lines of the file:
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@@
   )
   (layers
-    (0 F.Cu signal hide)
-    (31 B.Cu signal hide)
+    (0 F.Cu signal)
+    (31 B.Cu signal)
     (33 F.Adhes user)
     (35 F.Paste user)
@@
   (gr_line (start 99.904805 135.900923) (end 99.904805 149.901403) (layer Eco1.User) (width 0.1))
   (gr_line (start 85.905315 135.900923) (end 99.904805 135.900923) (layer Eco1.User) (width 0.1))
-  (gr_line (start 85.725 116.68125) (end 85.725 188.11875) (angle 90) (layer Edge.Cuts) (width 0.15))
-  (gr_line (start 102.39375 116.68125) (end 85.725 116.68125) (angle 90) (layer Edge.Cuts) (width 0.15))
+  (gr_line (start 87.025 116.68125) (end 87.025 188.11875) (angle 90) (layer Edge.Cuts) (width 0.15))
+  (gr_line (start 102.39375 116.68125) (end 87.025 116.68125) (angle 90) (layer Edge.Cuts) (width 0.15))
   (gr_line (start 102.39375 146.446875) (end 102.39375 116.68125) (angle 90) (layer Edge.Cuts) (width 0.15))
   (gr_line (start 111.91875 146.446875) (end 102.39375 146.446875) (angle 90) (layer Edge.Cuts) (width 0.15))
@@
   (gr_line (start 361.95 116.68125) (end 111.91875 116.68125) (angle 90) (layer Edge.Cuts) (width 0.15))
   (gr_line (start 361.95 188.11875) (end 361.95 116.68125) (angle 90) (layer Edge.Cuts) (width 0.15))
-  (gr_line (start 85.725 188.11875) (end 361.95 188.11875) (angle 90) (layer Edge.Cuts) (width 0.15))
+  (gr_line (start 87.025 188.11875) (end 361.95 188.11875) (angle 90) (layer Edge.Cuts) (width 0.15))
   (gr_line (start 265.2522 185.07141) (end 265.2522 187.981818) (layer Dwgs.User) (width 0.1))
   (gr_line (start 336.62109 115.806224) (end 350.62109 115.806224) (layer Dwgs.User) (width 0.1))
